File: 5C/PEPiS/pr7-8/kicad/pr7-8.kicad_sch (KiCad schematic)
At the start: 4 parts, among them J1 Conn_01x02, U1 STM32F103C8Tx

Commit message: feat(pr7-8): canonical schematic cleanup plus rebuilt report
Schematic: title No4 to #4, PWR1/PWR2 refs hidden. ERC 0/0,
connectivity unchanged. Report rebuilt from .gost-report
sources (now tracked for reproduction), figures re-exported,
docx plus pdf refreshed.
Other:
- note added: "Практическая работа #4. USART1 STM32F103C8, вариант 4"
- note removed: "Практическая работа №4. USART1 STM32F103C8, вариант 4"
- title: Практическая работа №4. USART1 STM32F103C8, вариант 4 -> Практическая работа #4. USART1 STM32F103C8, вариант 4
Changed lines of the file:
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@@
 	(paper "A4")
 	(title_block
-		(title "Практическая работа №4. USART1 STM32F103C8, вариант 4")
+		(title "Практическая работа #4. USART1 STM32F103C8, вариант 4")
 	)
 	(no_connect
@@
 		(property "Reference" "PWR2"
 			(at 116.84 73.406 0)
+			(hide yes)
 			(show_name no)
 			(do_not_autoplace no)
@@
 		(property "Reference" "PWR1"
 			(at 121.92 73.406 0)
+			(hide yes)
 			(show_name no)
 			(do_not_autoplace no)
@@
 		(at 96.52 67.31)
 	)
-	(text "Практическая работа №4. USART1 STM32F103C8, вариант 4"
+	(text "Практическая работа #4. USART1 STM32F103C8, вариант 4"
 		(exclude_from_sim no)
 		(at 55.88 43.18 0)
